File: fabrication/jlcpcb/source/hardware/FC_REV_A.kicad_sch (KiCad schematic)
At the start: 0 parts

Commit message: docs: publish neutral engineering source, manufacturing and portfolio overview
Other:
- company: FC DRONE PROJECT -> Desan Vasu
- title: FC_REV_A Flight Controller -> Flight Controller V1
